File: hardware/CC1101/CC1101ArduinoShield/CC1101-1190EM_Adapter_V3.00.brd (EAGLE design)
At the start: 14 parts, among them J1 20021121-00010T4LF, J2 20021121-00010T4LF, U2 RT9164A

Commit message: Update
Parts:
- added C3, C4: 33pF, eagle-ltspice:C0805
- C13, C14, C15, C16, C17, C18, C19: value 82pF -> 33pF
Connections:
- new net LNA_EN: C4.1, J1.P$7, U$1.P$2
- new net PA_EN: C15.1, C3.1, J1.P$3, U$1.P$3
- net CS: now also C19.1; no longer C18.1
- net GDO0: now also U$1.P$5
- net GDO2: no longer C15.1
- net GND: now also C3.2, C4.2; no longer J1.P$11, J1.P$13, J1.P$15, J1.P$17, J1.P$2, J1.P$3, J1.P$4, J1.P$5, J1.P$6, J1.P$7, J1.P$8, J1.P$9, J2.P$1, J2.P$10, J2.P$11, J2.P$12, J2.P$13, J2.P$14, J2.P$15, J2.P$16, J2.P$17, J2.P$18, J2.P$19, J2.P$20, J2.P$3, J2.P$4, J2.P$5, J2.P$6, J2.P$8
- net SCLK: now also C18.1; no longer C19.1
- net SI: now also C16.1; no longer C17.1
- net SO: now also C17.1; no longer C16.1
