File: hardware/CC1101/CC1101ArduinoShield/temp.sch (EAGLE design)
At the start: 16 parts, among them J1 20021121-00010T4LF, J2 20021121-00010T4LF, U2 RT9164A

Commit message: Update
Parts:
- removed C3, C4: 33pF, eagle-ltspice:C
- removed VIA89: GND_VIA_NO_THERMAL, fhmechanical:GND_VIA_NO_THERMAL
- added C11: 82pF, eagle-ltspice:C
- added VIA1, VIA10, VIA11, VIA12, VIA13, VIA14, VIA15, VIA16, VIA17, VIA18, VIA19, VIA2, VIA20, VIA21, VIA22, VIA23, VIA24, VIA25, VIA26, VIA27, VIA28, VIA29, VIA3, VIA30, VIA31, VIA32, VIA33, VIA34, VIA35, VIA36, VIA37, VIA38, VIA39, VIA4, VIA40, VIA41, VIA42, VIA43, VIA44, VIA45, VIA46, VIA47, VIA48, VIA49, VIA5, VIA50, VIA51, VIA52, VIA53, VIA54, VIA55, VIA56, VIA57, VIA58, VIA59, VIA6, VIA60, VIA61, VIA62, VIA63, VIA64, VIA65, VIA66, VIA67, VIA68, VIA69, VIA7, VIA70, VIA71, VIA72, VIA73, VIA74, VIA75, VIA76, VIA77, VIA78, VIA79, VIA8, VIA80, VIA81, VIA82, VIA83, VIA84, VIA85, VIA86, VIA87, VIA88, VIA9: GND_VIA_NO_THERMAL, fhmechanical:GND_VIA_NO_THERMAL
- C13, C14, C15, C16, C17, C18, C19: value 33pF -> 82pF
Connections:
- removed net LNA_EN: C4.1, J1.7, U$1.D8
- removed net PA_EN: C15.1, C3.1, J1.3, U$1.D7
- net CS: now also C18.1; no longer C19.1
- net GDO0: no longer U$1.D5
- net GDO2: now also C15.1
- net GND: now also C11.1, J1.11, J1.13, J1.15, J1.17, J1.2, J1.3, J1.4, J1.5, J1.6, J1.7, J1.8, J1.9, J2.1, J2.10, J2.11, J2.12, J2.13, J2.14, J2.15, J2.16, J2.17, J2.18, J2.19, J2.20, J2.3, J2.4, J2.5, J2.6, J2.8, VIA1.1, VIA10.1, VIA11.1, VIA12.1, VIA13.1, VIA14.1, VIA15.1, VIA16.1, VIA17.1, VIA18.1, VIA19.1, VIA2.1, VIA20.1, VIA21.1, VIA22.1, VIA23.1, VIA24.1, VIA25.1, VIA26.1, VIA27.1, VIA28.1, VIA29.1, VIA3.1, VIA30.1, VIA31.1, VIA32.1, VIA33.1, VIA34.1, VIA35.1, VIA36.1, VIA37.1, VIA38.1, VIA39.1, VIA4.1, VIA40.1, VIA41.1, VIA42.1, VIA43.1, VIA45.1, VIA46.1, VIA47.1, VIA48.1, VIA49.1, VIA5.1, VIA50.1, VIA51.1, VIA52.1, VIA53.1, VIA54.1, VIA55.1, VIA56.1, VIA57.1, VIA58.1, VIA59.1, VIA6.1, VIA60.1, VIA61.1, VIA62.1, VIA63.1, VIA64.1, VIA65.1, VIA66.1, VIA67.1, VIA68.1, VIA69.1, VIA7.1, VIA70.1, VIA71.1, VIA72.1, VIA73.1, VIA74.1, VIA75.1, VIA76.1, VIA77.1, VIA78.1, VIA79.1, VIA8.1, VIA80.1, VIA81.1, VIA82.1, VIA83.1, VIA84.1, VIA85.1, VIA86.1, VIA87.1, VIA88.1, VIA9.1; no longer C16.2, C3.2, C4.2
- net SCLK: now also C19.1; no longer C18.1
- net SI: now also C17.1; no longer C16.1
- net SO: now also C16.1; no longer C17.1
- net VIN: now also C11.2
Other:
- moved on the sheet: C1, C13, C14, C15, C16, C17, C18, C19, C2, J2, U2
