File: hardware/XTend/CommPositionDev/XtendTeensy.sch (EAGLE design)
At the start: 43 parts, among them J1 POWER_JACK, J2 HIROSE_DM3CS-SF, J3 JST_SM05B, SW1 SPDT_RA_3A, U1 TXB0108PWR, U2 5510003828F, U3 LM60, U4 COPERNICUS_II_DIP, U5 TEENSY_3.X, U6 7805T

Commit message: Update to state of XTendTeensy at move to FHComm repo
Parts:
- removed U1: TXB0108PWR, adafruit-fh:TXB0108PWR
- added U7: TXB0108PWR, adafruit-fh:TXB0108PWR
- C11: value 30pF -> 0.22uF
- R2: value (none) -> 10k
- SHLD3: value BMI-S-2XX1 -> BMI-S-2XX4; device fhmechanical:BMI-S-2XX1 -> fhmechanical:BMI-S-2XX4
- SHLD4: value BMI-S-2XX1 -> BMI-S-2XX5; device fhmechanical:BMI-S-2XX1 -> fhmechanical:BMI-S-2XX5
Connections:
- removed net N$15: U1.A1, U5.6
- removed net N$23: U1.A4, U5.15/A1
- removed net N$24: U1.A5, U5.16/A2
- removed net N$25: U1.A3, U5.10
- removed net N$26: U1.A6, U5.17/A3
- removed net N$4: U1.A2, U5.9
- removed net N$6: U1.A8, U5.18/A4
- removed net N$9: U1.A7, U5.19/A5
- net 3.3V: no longer U1.VCCA
- net 5.0V: now also A1.SHDN*; no longer U1.VCCB
- net GND: no longer A1.SHDN*, U1.GND
- net N$11: now also U5.16/A2; no longer U1.B5
- net N$12: now also U5.6; no longer U1.B1
- net N$13: now also U5.15/A1; no longer U1.B4
- net N$14: now also U5.17/A3; no longer U1.B6
- net N$5: now also U5.10; no longer U1.B3
- net N$8: now also U5.9; no longer U1.B2
- net SCL: now also U5.19/A5; no longer U1.B7
- net SDA: now also U5.18/A4; no longer U1.B8
Other:
- moved on the sheet: U6
